Commit message: Noetic Version
Updated version with 3 boxes, colors and variable shapes

File: urdf/blue_box.urdf (robot description, URDF)
Before this commit: robot red_box, 1 links, 0 joints
Links:
- link base_link: geometry collision box size=0.1 0.075 0.025; visual box size=0.1 0.075 0.025

File: urdf/conveyor_belt.urdf (robot description, URDF)
Before this commit: robot conveyor_belt, 2 links, 1 joints
Links:
- link base_link: geometry collision box size=5 0.65 0.2; visual box size=5 0.65 0.2

File: urdf/green_box.urdf (robot description, URDF)
Before this commit: robot red_box, 1 links, 0 joints
Links:
- link base_link: geometry collision box size=0.1 0.1 0.025; visual box size=0.1 0.1 0.025
